File: digit/pcb/glove/esp32/esp32.kicad_sch (KiCad schematic)
At the start: 68 parts, among them IC1 MDBT53-P1M, IC2 LTC3119EFE#PBF, IC3 DRV2605LDGSR, IC4 DRV2605LDGSR, IC5 TCA9546ADR, J1 Conn_02x05_Odd_Even, J10 Conn_01x03_Pin, J11 Conn_01x02_Pin, J12 Conn_01x02_Pin, J13 Conn_01x05_Pin, J14 Conn_01x02_Pin, J15 Conn_01x01_Pin, J16 Conn_01x02_Pin, J2 Conn_01x02_Pin, J3 Conn_01x02_Pin, J4 Conn_01x02_Pin, J5 Conn_01x02_Pin, J6 Conn_01x02_Pin, J7 Conn_01x02_Pin, J8 Conn_01x02_Pin, J9 Conn_01x02_Pin, Y1 FC-135R_32.7680KA-AG0

Commit message: Changed directory names to be proper
Parts:
- removed IC1: MDBT53-P1M, MDBT53-P1M:MDBT53P1M, symbol MDBT53-P1M:MDBT53-P1M
- removed IC2: LTC3119EFE#PBF, LTC3119EFE#PBF:SOP65P640X120-29N, symbol LITC3119:LTC3119EFE#PBF
- removed IC3, IC4: DRV2605LDGSR, DRV2605LDGSR:SOP50P490X110-10N, symbol TI DRV2605LDGSR:DRV2605LDGSR
- removed IC5: TCA9546ADR, TCA9546ADR:SOIC127P600X175-16N, symbol TCA9546ADR:TCA9546ADR
- removed J1: Conn_02x05_Odd_Even, Connector_PinHeader_2.54mm:PinHeader_2x05_P2.54mm_Vertical, symbol Connector_Generic:Conn_02x05_Odd_Even
- removed J10: Conn_01x03_Pin, Connector_PinHeader_2.54mm:PinHeader_1x03_P2.54mm_Vertical, symbol Connector:Conn_01x03_Pin
- removed J11, J16: Conn_01x02_Pin, Connector_PinHeader_2.54mm:PinHeader_1x02_P2.54mm_Vertical, symbol Connector:Conn_01x02_Pin
- removed J13: Conn_01x05_Pin, Connector_PinHeader_2.54mm:PinHeader_1x05_P2.54mm_Vertical, symbol Connector:Conn_01x05_Pin
- removed J15: Conn_01x01_Pin, Connector_PinHeader_2.54mm:PinHeader_1x01_P2.54mm_Vertical, symbol Connector:Conn_01x01_Pin
- removed J4, J7: Conn_01x02_Pin, Connector_Wire:SolderWire-0.5sqmm_1x02_P4.6mm_D0.9mm_OD2.1mm, symbol Connector:Conn_01x02_Pin
- removed Y1: FC-135R_32.7680KA-AG0, FC-135R_32.768KA-AGO:XTAL_FC-135R_32.7680KA-AG0, symbol FC-135R 32.7680KA-AG0:FC-135R_32.7680KA-AG0
- added C11: 470pF, Capacitor_SMD:C_0805_2012Metric_Pad1.18x1.45mm_HandSolder, symbol Device:C_Small
- added IC1, IC2: DRV2605LDGSR, DRV2605LDGSR:SOP50P490X110-10N, symbol TI DRV2605LDGSR:DRV2605LDGSR
- added IC3: LTC3119EFE#PBF, LTC3119EFE#PBF:SOP65P640X120-29N, symbol LITC3119:LTC3119EFE#PBF
- added IC4: TCA9546ADR, TCA9546ADR:SOIC127P600X175-16N, symbol TCA9546ADR:TCA9546ADR
- added J1: Conn_01x02_Pin, Connector_JST:JST_PH_S2B-PH-K_1x02_P2.00mm_Horizontal, symbol Connector:Conn_01x02_Pin
- added J10: USB_C_Receptacle_USB2.0_16P, Connector_USB:USB_C_Receptacle_GCT_USB4105-xx-A_16P_TopMnt_Horizontal, symbol Connector:USB_C_Receptacle_USB2.0_16P
- added J11: Conn_01x05_Pin, Connector_PinHeader_2.54mm:PinHeader_1x05_P2.54mm_Vertical, symbol Connector:Conn_01x05_Pin
- added J13: Conn_01x02_Pin, Connector_PinHeader_2.54mm:PinHeader_1x02_P2.54mm_Vertical, symbol Connector:Conn_01x02_Pin
- added J15, J17: Conn_01x02_Pin, Connector_Wire:SolderWire-0.5sqmm_1x02_P4.6mm_D0.9mm_OD2.1mm, symbol Connector:Conn_01x02_Pin
- added J18: Conn_01x04_Pin, Connector_PinHeader_2.54mm:PinHeader_1x04_P2.54mm_Vertical, symbol Connector:Conn_01x04_Pin
- added J4: Conn_01x03_Pin, Connector_PinHeader_2.54mm:PinHeader_1x03_P2.54mm_Vertical, symbol Connector:Conn_01x03_Pin
- added J7: Conn_01x01_Pin, Connector_PinHeader_2.54mm:PinHeader_1x01_P2.54mm_Vertical, symbol Connector:Conn_01x01_Pin
- added R24: 1k, Resistor_SMD:R_0805_2012Metric_Pad1.20x1.40mm_HandSolder, symbol Device:R_Small
- added R26, R8: 10k, Resistor_SMD:R_0805_2012Metric_Pad1.20x1.40mm_HandSolder, symbol Device:R_Small
- added SW1: SW_Push, Button_Switch_SMD:SW_SPST_PTS645, symbol Switch:SW_Push
- added U1: ESP32-S3-WROOM-1, RF_Module:ESP32-S3-WROOM-1, symbol RF_Module:ESP32-S3-WROOM-1
- C1: value 0.1µF -> 10µF
- C10: value 4.7µF -> 100nF
- C12: value 1µF -> 150µF; footprint Capacitor_SMD:C_0805_2012Metric_Pad1.18x1.45mm_HandSolder -> Capacitor_SMD:C_Elec_10x10.2
- C13: value 1µF -> 0.1µF
- C14, C15: value 1µF -> 100nF
- C16: value 0.1µF -> 100nF
- C19, C20: value 100nF -> 0.1uF
- C2: value 0.1µF -> 1µF
- C21: value 100nF -> 22uF
- C3: value 10µF -> 1µF
- C4: value 4.7µF -> 0.1µF
- C5: value 470pF -> 4.7µF
- C6: value 150µF -> 100nF; footprint Capacitor_SMD:C_Elec_10x10.2 -> Capacitor_SMD:C_0805_2012Metric_Pad1.18x1.45mm_HandSolder
- C7, C8: value 100nF -> 1µF
- C9: value 2.2µF -> 0.1µF
- J12: footprint Connector_PinHeader_2.54mm:PinHeader_1x02_P2.54mm_Vertical -> Connector_Wire:SolderWire-0.5sqmm_1x02_P4.6mm_D0.9mm_OD2.1mm
- J6: footprint Connector_Wire:SolderWire-0.5sqmm_1x02_P4.6mm_D0.9mm_OD2.1mm -> Connector_PinHeader_2.54mm:PinHeader_1x02_P2.54mm_Vertical
- J9: footprint Connector_JST:JST_PH_S2B-PH-K_1x02_P2.00mm_Horizontal -> Connector_PinHeader_2.54mm:PinHeader_1x02_P2.54mm_Vertical
- R10: value 22k -> 100k
- R11, R13, R15, R19: value 1k -> 22k
- R12, R14: value 22k -> 1k
- R16, R18: value 22k -> 5.1k
- R20: value 10k -> 1k
- R23: value 10k -> 22k
- R3: value 52.3k -> 10k
- R4: value 316k -> 10k
- R5: value 100k -> 10k
- R6: value 10k -> 52.3k
- R9: value 10k -> 316k
Connections:
- net +3.7V: now also J1.1 (Pin_1); no longer J9.1 (Pin_1)
- net BB_3V3: now also C12.1, R9.2, IC3.6 (PVOUT_1), IC3.7 (PVOUT_2), J4.3 (Pin_3); no longer C6.1, R4.2
- net EXT_3V3: now also J6.2 (Pin_2)
- net FLEX1_ADC: now also C14.1, R12.2, J11.5 (Pin_5), U1.39 (IO1); no longer C17.1, R11.2
- net FLEX2_ADC: now also C15.1, R14.2, J11.4 (Pin_4), U1.38 (IO2); no longer C18.1, R13.2
- net FLEX3_ADC: now also C16.1, R17.2, J11.3 (Pin_3), U1.15 (IO3); no longer C21.1, R19.2
- net FLEX4_ADC: now also C17.1, R20.2, J11.2 (Pin_2), U1.4 (IO4); no longer C19.1, R15.2
- net FLEX5_ADC: now also C18.1, J11.1 (Pin_1), R24.2, U1.5 (IO5); no longer C20.1, R17.2
- net GND: now also C1.2, C13.1, C16.2, C2.2, C6.1, C8.2, J12.2 (Pin_2), J14.1 (Pin_1), J6.1 (Pin_1), R10.1, R16.1, R18.1, C11.2, IC1.3 (SDA), IC1.7 (OUT+), IC2.3 (SDA), IC2.7 (OUT+), IC3.14 (SGND), IC3.20 (PGND_3), IC3.25 (PGND_4), IC3.28 (PWM/SYNC), IC3.29 (PGND_5), IC3.4 (PGND_1), IC3.9 (PGND_2), IC4.1 (A0), IC4.13 (A2), IC4.2 (A1), IC4.8 (GND), J1.2 (Pin_2), J10.A1 (GND), J10.A12 (GND), J10.B1 (GND), J10.B12 (GND), J10.S1 (SHIELD), J15.2 (Pin_2), J17.2 (Pin_2), J18.1 (Pin_1), SW1.1, U1.1 (GND), U1.40 (GND), U1.41 (GND); no longer C13.2, C16.1, C4.2, C6.2, C8.1, C9.2, J6.2 (Pin_2), J9.2 (Pin_2), R5.1
- net HAPTIC_DRIVER1_EN: now also IC1.6 (VDD/NC), J13.2 (Pin_2); no longer J14.2 (Pin_2)
- net HAPTIC_DRIVER2_EN: now also IC2.6 (VDD/NC), J13.1 (Pin_1); no longer J14.1 (Pin_1)
- net I2C_SCL: now also J9.1 (Pin_1), R21.2, IC4.14 (SCL), U1.17 (IO9); no longer J12.1 (Pin_1), R6.2
- net I2C_SDA: now also J9.2 (Pin_2), R22.2, IC4.15 (SDA), U1.12 (IO8); no longer J12.2 (Pin_2), R7.2
- net IMU_INT1: now also J7.1 (Pin_1), U1.18 (IO10)
- net SYS_3V3: now also C13.2, C2.1, C20.1, C21.1, C3.1, C6.2, R11.1, R13.1, R15.1, R19.1, R3.1, R4.1, R5.1, IC1.1 (REG), IC1.5 (EN), IC2.1 (REG), IC2.5 (EN), IC4.16 (VCC), J18.4 (Pin_4), J4.2 (Pin_2), R26.2, R8.2, U1.2 (3V3); no longer C14.1, C15.1, C16.2, C7.1, C8.2, C9.1, R10.1, R12.1, R14.1, R16.1, R18.1, R20.1, R6.1, R9.2
- net UART_RX: now also J18.2 (Pin_2), U1.36 (RXD0)
- net UART_TX: now also J18.3 (Pin_3), U1.37 (TXD0)
- net at R16.2: now also J10.B5 (CC2); no longer R17.1
- net at R2.2: now also IC3.17 (RT)
- net at C5.1: now also IC3.11 (SVCC), IC3.15 (MPPC), IC3.16 (VCC); no longer R3.1
- net at R3.2: now also IC2.8 (GND), IC4.4 (SD0)
- net at F2.2: now also J4.1 (Pin_1)
- net at F1.1, R1.1: now also C1.1, IC3.19 (VIN), IC3.22 (PVIN_1), IC3.23 (PVIN_2); no longer C3.1
- net at J2.2 (Pin_2): now also IC1.4 (IN/TRIG)
- net at J2.1 (Pin_1): now also IC1.2 (SCL)
- net at R23.2: now also J17.1 (Pin_1), R24.1
- net at C4.1: now also L1.2, IC3.21 (SW1_1), IC3.24 (SW1_2)
- net at R5.2: now also IC2.9 (OUT-), IC4.5 (SC0); no longer R4.1
- net at R1.2: now also IC3.18 (RUN)
- net at L1.1: now also C9.1, IC3.5 (SW2_1), IC3.8 (SW2_2); no longer C2.1
- net at J3.2 (Pin_2): now also IC2.4 (IN/TRIG)
- net at J3.1 (Pin_1): now also IC2.2 (SCL)
- net at R9.1: now also R10.2, IC3.12 (FB)
- new net: J15.1 (Pin_1), R19.2, R20.1
- new net: J10.A5 (CC1), R18.2
- new net: IC4.3 (~{RESET}), R8.1
- new net: IC1.8 (GND), IC4.6 (SD1), R4.2
- new net: IC1.9 (OUT-), IC4.7 (SC1), R7.2
- new net: C7.1, IC2.10 (VDD)
- new net: C8.1, IC1.10 (VDD)
- new net: J12.1 (Pin_1), R15.2, R17.1
- new net: J5.1 (Pin_1), R11.2, R12.1
- new net: C11.1, R6.1
- new net: IC3.13 (VC), R6.2
- new net: C9.2, IC3.3 (BST2)
- new net: J8.1 (Pin_1), R13.2, R14.1
- new net: J10.A4 (VBUS), J10.A9 (VBUS), J10.B4 (VBUS), J10.B9 (VBUS)
- new net: C4.2, IC3.26 (BST1)
- new net BOOT: J14.2 (Pin_2), U1.27 (IO0)
- new net Dn: J10.A7 (D-), J10.B7 (D-), U1.13 (USB_D-)
- new net Dp: J10.A6 (D+), J10.B6 (D+), U1.14 (USB_D+)
- new net EN: C19.1, R26.1, SW1.2, U1.3 (EN)
- no-connect marks 59 -> 39
