File: digit/pcb/glove/nrf5340/nrf5340.kicad_sch (KiCad schematic)
At the start: 73 parts, among them IC1 DRV2605LDGSR, IC2 DRV2605LDGSR, IC3 LTC3119EFE#PBF, IC4 TCA9546ADR, J1 Conn_01x02_Pin, J10 USB_C_Receptacle_USB2.0_16P, J11 Conn_01x05_Pin, J12 Conn_01x02_Pin, J13 Conn_01x02_Pin, J14 Conn_01x02_Pin, J15 Conn_01x02_Pin, J17 Conn_01x02_Pin, J18 Conn_01x04_Pin, J2 Conn_01x02_Pin, J3 Conn_01x02_Pin, J4 Conn_01x03_Pin, J5 Conn_01x02_Pin, J6 Conn_01x02_Pin, J7 Conn_01x01_Pin, J8 Conn_01x02_Pin, J9 Conn_01x02_Pin, SW1 SW_Push, U1 ESP32-S3-WROOM-1

Commit message: Changed directory names to be proper
Parts:
- removed C11: 470pF, Capacitor_SMD:C_0805_2012Metric_Pad1.18x1.45mm_HandSolder, symbol Device:C_Small
- removed IC1, IC2: DRV2605LDGSR, DRV2605LDGSR:SOP50P490X110-10N, symbol TI DRV2605LDGSR:DRV2605LDGSR
- removed IC3: LTC3119EFE#PBF, LTC3119EFE#PBF:SOP65P640X120-29N, symbol LITC3119:LTC3119EFE#PBF
- removed IC4: TCA9546ADR, TCA9546ADR:SOIC127P600X175-16N, symbol TCA9546ADR:TCA9546ADR
- removed J1: Conn_01x02_Pin, Connector_JST:JST_PH_S2B-PH-K_1x02_P2.00mm_Horizontal, symbol Connector:Conn_01x02_Pin
- removed J10: USB_C_Receptacle_USB2.0_16P, Connector_USB:USB_C_Receptacle_GCT_USB4105-xx-A_16P_TopMnt_Horizontal, symbol Connector:USB_C_Receptacle_USB2.0_16P
- removed J11: Conn_01x05_Pin, Connector_PinHeader_2.54mm:PinHeader_1x05_P2.54mm_Vertical, symbol Connector:Conn_01x05_Pin
- removed J13: Conn_01x02_Pin, Connector_PinHeader_2.54mm:PinHeader_1x02_P2.54mm_Vertical, symbol Connector:Conn_01x02_Pin
- removed J15, J17: Conn_01x02_Pin, Connector_Wire:SolderWire-0.5sqmm_1x02_P4.6mm_D0.9mm_OD2.1mm, symbol Connector:Conn_01x02_Pin
- removed J18: Conn_01x04_Pin, Connector_PinHeader_2.54mm:PinHeader_1x04_P2.54mm_Vertical, symbol Connector:Conn_01x04_Pin
- removed J4: Conn_01x03_Pin, Connector_PinHeader_2.54mm:PinHeader_1x03_P2.54mm_Vertical, symbol Connector:Conn_01x03_Pin
- removed J7: Conn_01x01_Pin, Connector_PinHeader_2.54mm:PinHeader_1x01_P2.54mm_Vertical, symbol Connector:Conn_01x01_Pin
- removed R24: 1k, Resistor_SMD:R_0805_2012Metric_Pad1.20x1.40mm_HandSolder, symbol Device:R_Small
- removed R26, R8: 10k, Resistor_SMD:R_0805_2012Metric_Pad1.20x1.40mm_HandSolder, symbol Device:R_Small
- removed SW1: SW_Push, Button_Switch_SMD:SW_SPST_PTS645, symbol Switch:SW_Push
- removed U1: ESP32-S3-WROOM-1, RF_Module:ESP32-S3-WROOM-1, symbol RF_Module:ESP32-S3-WROOM-1
- added IC1: MDBT53-P1M, MDBT53-P1M:MDBT53P1M, symbol MDBT53-P1M:MDBT53-P1M
- added IC2: LTC3119EFE#PBF, LTC3119EFE#PBF:SOP65P640X120-29N, symbol LITC3119:LTC3119EFE#PBF
- added IC3, IC4: DRV2605LDGSR, DRV2605LDGSR:SOP50P490X110-10N, symbol TI DRV2605LDGSR:DRV2605LDGSR
- added IC5: TCA9546ADR, TCA9546ADR:SOIC127P600X175-16N, symbol TCA9546ADR:TCA9546ADR
- added J1: Conn_02x05_Odd_Even, Connector_PinHeader_2.54mm:PinHeader_2x05_P2.54mm_Vertical, symbol Connector_Generic:Conn_02x05_Odd_Even
- added J10: Conn_01x03_Pin, Connector_PinHeader_2.54mm:PinHeader_1x03_P2.54mm_Vertical, symbol Connector:Conn_01x03_Pin
- added J11, J16: Conn_01x02_Pin, Connector_PinHeader_2.54mm:PinHeader_1x02_P2.54mm_Vertical, symbol Connector:Conn_01x02_Pin
- added J13: Conn_01x05_Pin, Connector_PinHeader_2.54mm:PinHeader_1x05_P2.54mm_Vertical, symbol Connector:Conn_01x05_Pin
- added J15: Conn_01x01_Pin, Connector_PinHeader_2.54mm:PinHeader_1x01_P2.54mm_Vertical, symbol Connector:Conn_01x01_Pin
- added J4, J7: Conn_01x02_Pin, Connector_Wire:SolderWire-0.5sqmm_1x02_P4.6mm_D0.9mm_OD2.1mm, symbol Connector:Conn_01x02_Pin
- added Y1: FC-135R_32.7680KA-AG0, FC-135R_32.768KA-AGO:XTAL_FC-135R_32.7680KA-AG0, symbol FC-135R 32.7680KA-AG0:FC-135R_32.7680KA-AG0
- C1: value 10µF -> 0.1µF
- C10: value 100nF -> 4.7µF
- C12: value 150µF -> 1µF; footprint Capacitor_SMD:C_Elec_10x10.2 -> Capacitor_SMD:C_0805_2012Metric_Pad1.18x1.45mm_HandSolder
- C13: value 0.1µF -> 1µF
- C14, C15: value 100nF -> 1µF
- C16: value 100nF -> 0.1µF
- C19, C20: value 0.1uF -> 100nF
- C2: value 1µF -> 0.1µF
- C21: value 22uF -> 100nF
- C3: value 1µF -> 10µF
- C4: value 0.1µF -> 4.7µF
- C5: value 4.7µF -> 470pF
- C6: value 100nF -> 150µF; footprint Capacitor_SMD:C_0805_2012Metric_Pad1.18x1.45mm_HandSolder -> Capacitor_SMD:C_Elec_10x10.2
- C7, C8: value 1µF -> 100nF
- C9: value 0.1µF -> 2.2µF
- J12: footprint Connector_Wire:SolderWire-0.5sqmm_1x02_P4.6mm_D0.9mm_OD2.1mm -> Connector_PinHeader_2.54mm:PinHeader_1x02_P2.54mm_Vertical
- J6: footprint Connector_PinHeader_2.54mm:PinHeader_1x02_P2.54mm_Vertical -> Connector_Wire:SolderWire-0.5sqmm_1x02_P4.6mm_D0.9mm_OD2.1mm
- J9: footprint Connector_PinHeader_2.54mm:PinHeader_1x02_P2.54mm_Vertical -> Connector_JST:JST_PH_S2B-PH-K_1x02_P2.00mm_Horizontal
- R10: value 100k -> 22k
- R11, R13, R15, R19: value 22k -> 1k
- R12, R14: value 1k -> 22k
- R16, R18: value 5.1k -> 22k
- R20: value 1k -> 10k
- R23: value 22k -> 10k
- R3: value 10k -> 52.3k
- R4: value 10k -> 316k
- R5: value 10k -> 100k
- R6: value 52.3k -> 10k
- R9: value 316k -> 10k
Connections:
- net BOOT is gone; now on net HAPTIC_DRIVER1_EN: J14.2 (Pin_2)
- net EN is gone; now on net FLEX4_ADC: C19.1
- net +3.7V: now also J9.1 (Pin_1)
- net BB_3V3: now also C6.1, R4.2, IC2.6 (PVOUT_1), IC2.7 (PVOUT_2), J10.3 (Pin_3); no longer C12.1, R9.2
- net EXT_3V3: now also J11.2 (Pin_2); no longer J6.2 (Pin_2)
- net FLEX1_ADC: now also C17.1, R11.2, IC1.9 (P0.25), J13.5 (Pin_5); no longer C14.1, R12.2
- net FLEX2_ADC: now also C18.1, R13.2, IC1.60 (P0.28), J13.4 (Pin_4); no longer C15.1, R14.2
- net FLEX3_ADC: now also C21.1, R19.2, IC1.39 (P0.05), J13.3 (Pin_3); no longer C16.1, R17.2
- net FLEX4_ADC: now also R15.2, IC1.35 (P0.06), J13.2 (Pin_2); no longer C17.1, R20.2
- net FLEX5_ADC: now also C20.1, R17.2, IC1.20 (P0.07), J13.1 (Pin_1); no longer C18.1
- net GND: now also C13.2, C16.1, C4.2, C6.2, C8.1, C9.2, J6.2 (Pin_2), J9.2 (Pin_2), R5.1, IC1.1 (GND_1), IC1.24 (GND_2), IC1.42 (GND_3), IC1.44 (VBUS), IC1.61 (GND_4), IC2.14 (SGND), IC2.20 (PGND_3), IC2.25 (PGND_4), IC2.28 (PWM/SYNC), IC2.29 (PGND_5), IC2.4 (PGND_1), IC2.9 (PGND_2), IC3.4 (IN/TRIG), IC3.8 (GND), IC4.4 (IN/TRIG), IC4.8 (GND), IC5.1 (A0), IC5.13 (A2), IC5.2 (A1), IC5.8 (GND), J1.3 (Pin_3), J1.5 (Pin_5), J11.1 (Pin_1), J4.2 (Pin_2), J7.2 (Pin_2); no longer C1.2, C13.1, C16.2, C2.2, C6.1, C8.2, J12.2 (Pin_2), J14.1 (Pin_1), J6.1 (Pin_1), R10.1, R16.1, R18.1
- net HAPTIC_DRIVER1_EN: now also IC1.7 (P0.26), IC3.5 (EN)
- net HAPTIC_DRIVER2_EN: now also J14.1 (Pin_1), IC1.62 (P0.23), IC4.5 (EN)
- net I2C_SCL: now also J12.1 (Pin_1), R6.2, IC1.33 (P1.02), IC5.14 (SCL); no longer J9.1 (Pin_1), R21.2
- net I2C_SDA: now also J12.2 (Pin_2), R7.2, IC1.31 (P1.03), IC5.15 (SDA); no longer J9.2 (Pin_2), R22.2
- net IMU_INT1: now also IC1.37 (P0.04), J15.1 (Pin_1)
- net SYS_3V3: now also C14.1, C15.1, C16.2, C7.1, C8.2, C9.1, R10.1, R12.1, R14.1, R16.1, R18.1, R20.1, R6.1, R9.2, IC1.38 (VDD), IC1.41 (VDDH), IC3.10 (VDD), IC3.6 (VDD/NC), IC4.10 (VDD), IC4.6 (VDD/NC), IC5.16 (VCC), J1.1 (Pin_1), J10.2 (Pin_2); no longer C13.2, C2.1, C20.1, C21.1, C3.1, C6.2, R11.1, R13.1, R15.1, R19.1, R3.1, R4.1, R5.1
- net UART_RX: now also IC1.29 (P0.08), J16.2 (Pin_2)
- net UART_TX: now also IC1.10 (P1.06), J16.1 (Pin_1)
- net at R9.1: now also IC5.3 (~{RESET}); no longer R10.2
- net at R16.2: now also R17.1, J7.1 (Pin_1)
- net at R18.2: now also J8.1 (Pin_1), R19.1
- net at R3.2: now also IC2.13 (VC)
- net at R5.2: now also R4.1, IC2.12 (FB)
- net at J3.1 (Pin_1): now also IC4.9 (OUT-)
- net at J3.2 (Pin_2): now also IC4.7 (OUT+)
- net at R23.2: now also IC4.2 (SCL), IC5.5 (SC0)
- net at F2.2: now also J10.1 (Pin_1)
- net at C5.1: now also R3.1
- net at L1.1: now also C2.1, IC2.5 (SW2_1), IC2.8 (SW2_2); no longer C9.1
- net at R2.2: now also IC2.17 (RT)
- net at F1.1, R1.1: now also C3.1, IC2.19 (VIN), IC2.22 (PVIN_1), IC2.23 (PVIN_2); no longer C1.1
- net at C4.1: now also IC2.11 (SVCC), IC2.15 (MPPC), IC2.16 (VCC); no longer L1.2
- net at J2.1 (Pin_1): now also IC3.9 (OUT-)
- net at J2.2 (Pin_2): now also IC3.7 (OUT+)
- net at R1.2: now also IC2.18 (RUN)
- new net: IC3.3 (SDA), IC5.6 (SD1), R21.2
- new net: IC3.2 (SCL), IC5.7 (SC1), R20.2
- new net: C12.1, IC3.1 (REG)
- new net: J5.1 (Pin_1), R12.2, R13.1
- new net: C1.1, IC2.21 (SW1_1), IC2.24 (SW1_2), L1.2
- new net: C1.2, IC2.26 (BST1)
- new net: C2.2, IC2.3 (BST2)
- new net: C13.1, IC4.1 (REG)
- new net: J6.1 (Pin_1), R14.2, R15.1
- new net: IC1.34 (P0.00/XL1), Y1.1
- new net: IC1.36 (P0.01/XL2), Y1.2
- new net: IC4.3 (SDA), IC5.4 (SD0), R22.2
- new net: J4.1 (Pin_1), R10.2, R11.1
- new net RESET: IC1.6 (RESET), J1.10 (Pin_10)
- new net SWDCLK: IC1.2 (SWDCLK), J1.4 (Pin_4)
- new net SWDIO: IC1.4 (SWDIO), J1.2 (Pin_2)
- no-connect marks 39 -> 59
